File: MetalBird_v2/MetalBird_v2.kicad_pro.kicad_pcb (KiCad board)
At the start: 2 copper layers, 38 x 38 mm, 71 parts, among them J1 Battery Conn, J10 VTX Conn, J2 SWD, J3 ESC1, J4 ESC2, J5 ESC3, J6 ESC4, J7 ELRS Reciver, J8 USB/UART DEBUG, J9 Camera Conn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

Commit message: Redesign: 4 in 1 ESC
- yet to route traces
Parts:
- removed J1: Battery Conn, Connector_JST:JST_PH_B2B-PH-K_1x02_P2.00mm_Vertical
- removed J4: ESC2, Connector_PinHeader_2.54mm:PinHeader_1x03_P2.54mm_Vertical
- removed J5: ESC3, Connector_PinHeader_2.54mm:PinHeader_1x03_P2.54mm_Vertical
- removed J6: ESC4, Connector_PinHeader_2.54mm:PinHeader_1x03_P2.54mm_Vertical
- J3: value ESC1 -> Conn_01x08; footprint Connector_PinHeader_2.54mm:PinHeader_1x03_P2.54mm_Vertical -> Connector_JST:JST_SH_BM08B-SRSS-TB_1x08-1MP_P1.00mm_Vertical
- moved J3 16.7 mm to (111.0, 93.0)
Connections:
- C1 pad 2: GND -> GBAT
- C10 pad 1: GND -> GBAT
- C12 pad 1: GND -> GBAT
- C14 pad 2: GND -> GBAT
- C15 pad 1: GND -> GBAT
- C16 pad 2: GND -> GBAT
- C17 pad 1: GND -> GBAT
- C18 pad 1: GND -> GBAT
- C19 pad 2: GND -> GBAT
- C1A1 pad 1: GND -> GBAT
- C2 pad 1: GND -> GBAT
- C20 pad 2: GND -> GBAT
- C21 pad 2: GND -> GBAT
- C22 pad 2: GND -> GBAT
- C23 pad 2: GND -> GBAT
- C24 pad 2: GND -> GBAT
- C25 pad 2: GND -> GBAT
- C26 pad 2: GND -> GBAT
- C2A1 pad 2: GND -> GBAT
- C3 pad 2: GND -> GBAT
- C4 pad 2: GND -> GBAT
- C5 pad 2: GND -> GBAT
- C6 pad 2: GND -> GBAT
- C7 pad 2: GND -> GBAT
- C8 pad 2: GND -> GBAT
- C9 pad 2: GND -> GBAT
- D1 pad 1: GND -> GBAT
- D2 pad 1: GND -> GBAT
- J10 pad 2: GND -> GBAT
- J2 pad 4: GND -> GBAT
- J3 pad 1: GND -> VBAT
- J3 pad 2: 5V -> GBAT
- J3 pad 3: Net-(J3-Pin_3) -> unconnected-(J3-Pin_3-Pad3)
- J7 pad 2: GND -> GBAT
- J8 pad 2: GND -> GBAT
- J9 pad 2: GND -> GBAT
- MP2331H1 pad 4: GND -> GBAT
- Q1 pad 3: Net-(J1-Pin_1) -> VBAT
- R12 pad 2: GND -> GBAT
- R2 pad 1: GND -> GBAT
- R8 pad 2: GND -> GBAT
- R9 pad 1: GND -> GBAT
- SW1 pad 1: GND -> GBAT
- U1 pad 23: GND -> GBAT
- U1 pad 29: Net-(J3-Pin_3) -> Net-(J3-Pin_5)
- U1 pad 30: Net-(J4-Pin_3) -> Net-(J3-Pin_6)
- U1 pad 31: Net-(J5-Pin_3) -> Net-(J3-Pin_7)
- U1 pad 32: Net-(J6-Pin_3) -> Net-(J3-Pin_8)
- U1 pad 35: GND -> GBAT
- U1 pad 47: GND -> GBAT
- U1 pad 49: GND -> GBAT
- U1 pad 8: GND -> GBAT
- U2 pad 1: GND -> GBAT
- U3 pad 1: GND -> GBAT
- U3 pad 11: GND -> GBAT
- U3 pad 18: GND -> GBAT
- U3 pad 9: GND -> GBAT
- U4 pad 1: GND -> GBAT
- U4 pad 7: GND -> GBAT
Routing:
- net Net-(J4-Pin_3): track 54.2 -> 0.00 mm, vias 5 -> 0
- net Net-(J3-Pin_6): track 0.00 -> 54.2 mm, vias 0 -> 5
- net Net-(J3-Pin_5): track 0.00 -> 35.4 mm, vias 0 -> 1
- net Net-(J3-Pin_3): track 35.4 -> 0.00 mm, vias 1 -> 0
- net Net-(J6-Pin_3): track 19.1 -> 0.00 mm, vias 5 -> 0
- net Net-(J3-Pin_8): track 0.00 -> 19.1 mm, vias 0 -> 5
- net Net-(J5-Pin_3): track 18.1 -> 0.00 mm, vias 3 -> 0
- net Net-(J3-Pin_7): track 0.00 -> 18.1 mm, vias 0 -> 3
- net Net-(J1-Pin_1): track 6.98 -> 0.00 mm
- net GBAT: track 0.00 -> 4.14 mm, vias 0 -> 32
- net GND: track 307.2 -> 303.1 mm, vias 32 -> 0
- added copper zone on B.Cu, net GBAT
- removed copper zone on B.Cu, net GND
