File: MetalBird_v2/MetalBird_v2.kicad_pro.kicad_sch (KiCad schematic)
At the start: 71 parts, among them J1 Battery Conn, J10 VTX Conn, J2 SWD, J3 ESC1, J4 ESC2, J5 ESC3, J6 ESC4, J7 ELRS Reciver, J8 USB/UART DEBUG, J9 Camera Conn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

Commit message: Redesign: 4 in 1 ESC
- yet to route traces
Parts:
- removed J1: Battery Conn, Connector_JST:JST_PH_B2B-PH-K_1x02_P2.00mm_Vertical, symbol Connector_Generic:Conn_01x02
- removed J3: ESC1, Connector_PinHeader_2.54mm:PinHeader_1x03_P2.54mm_Vertical, symbol Connector_Generic:Conn_01x03
- removed J4: ESC2, Connector_PinHeader_2.54mm:PinHeader_1x03_P2.54mm_Vertical, symbol Connector_Generic:Conn_01x03
- removed J5: ESC3, Connector_PinHeader_2.54mm:PinHeader_1x03_P2.54mm_Vertical, symbol Connector_Generic:Conn_01x03
- removed J6: ESC4, Connector_PinHeader_2.54mm:PinHeader_1x03_P2.54mm_Vertical, symbol Connector_Generic:Conn_01x03
- added J3: Conn_01x08, Connector_JST:JST_SH_BM08B-SRSS-TB_1x08-1MP_P1.00mm_Vertical, symbol Connector_Generic:Conn_01x08
Connections:
- net GND: now also J3.2 (Pin_2)
- net at U1.30 (PA9): now also J3.6 (Pin_6)
- net VBAT: now reaches Q1.3 (S)
- net VBAT: now also J3.1 (Pin_1)
- net at U1.31 (PA10): now also J3.7 (Pin_7)
- net at U1.29 (PA8): now also J3.5 (Pin_5)
- net at U1.32 (PA11): now also J3.8 (Pin_8)
- no-connect marks 20 -> 22

Commit message: Buck Converter change
Parts:
- removed C11: 1microF, Capacitor_SMD:C_0603_1608Metric, symbol Device:C
- removed C13: 10pF, Capacitor_SMD:C_0603_1608Metric, symbol Device:C
- removed C1A1: 0.1µF, Capacitor_SMD:C_0603_1608Metric, symbol Device:C
- removed C24: 100microF, Capacitor_SMD:C_1206_3216Metric, symbol Device:C_Polarized
- removed C7: 4.7nF, Capacitor_SMD:C_0603_1608Metric, symbol Device:C
- removed J2: SWD, Connector_PinHeader_2.54mm:PinHeader_1x04_P2.54mm_Vertical, symbol Connector_Generic:Conn_01x04
- removed J8: USB/UART DEBUG, Connector_PinHeader_2.54mm:PinHeader_1x04_P2.54mm_Vertical, symbol Connector_Generic:Conn_01x04
- removed MP2331H1: (no value), Package_TO_SOT_SMD:SOT-583-8, symbol Metal_bird_library:MP2331H
- removed R10: 300kΩ, Resistor_SMD:R_0603_1608Metric, symbol Device:R
- removed R18: 4.7kΩ, Resistor_SMD:R_0603_1608Metric, symbol Device:R
- removed R19: 18kΩ, Resistor_SMD:R_0603_1608Metric, symbol Device:R
- removed R20: 200, Resistor_SMD:R_0603_1608Metric, symbol Device:R
- removed R7: 22kΩ, Resistor_SMD:R_0603_1608Metric, symbol Device:R
- removed R9: 180Ω, Resistor_SMD:R_0603_1608Metric, symbol Device:R
- added AP62200WU-1: (no value), Package_TO_SOT_SMD:TSOT-23-6, symbol Metal_bird_library:AP62200WU-7
- added C2A2: 100µF, Capacitor_SMD:C_1206_3216Metric, symbol Device:C
- added J1: SWD, Connector_PinHeader_2.54mm:PinHeader_1x05_P2.54mm_Vertical, symbol Connector_Generic:Conn_01x05
- added J11: USB/UART DEBUG, Connector_PinHeader_2.54mm:PinHeader_1x03_P2.54mm_Vertical, symbol Connector_Generic:Conn_01x03
- C2: value 22µF -> 10µF
- C26: value 2.2nF -> 22µF; footprint Capacitor_SMD:C_0603_1608Metric -> Capacitor_SMD:C_1206_3216Metric
- C5: value 1nF -> 330nF; footprint Capacitor_SMD:C_0603_1608Metric -> (none)
- L1: value 2.2µH -> 3.3µH; footprint Inductor_SMD:L_Cenker_CKCS4018 -> Inductor_SMD:L_APV_ANR6045
- R1: value 300kΩ -> 47K; footprint Resistor_SMD:R_0603_1608Metric -> (none)
- R3: value 20ohm -> 10K; footprint Resistor_SMD:R_0603_1608Metric -> (none)
- R4: value 10kΩ -> 3K; footprint Resistor_SMD:R_0603_1608Metric -> (none)
- R5: value 7.5kΩ -> 3.3K; footprint Resistor_SMD:R_0603_1608Metric -> (none)
- Y1: footprint Crystal:Crystal_SMD_3225-4Pin_3.2x2.5mm -> Crystal:Crystal_SMD_5032-2Pin_5.0x3.2mm
Connections:
- net 3.3V: now also J1.2 (Pin_2)
- net 5V: now also C26.1, R1.1
- net 7.4V: now also AP62200WU-1.3 (VIN), AP62200WU-1.5 (EN), C2A2.1; no longer Q1.2 (G), R1.2, R8.1
- net GND: now also R3.1, AP62200WU-1.1 (GND), C2A2.2, J1.5 (Pin_5), J11.1 (Pin_1); no longer C26.2, C5.2
- net SWDCLK: now also J1.4 (Pin_4)
- net SWDIO: now also J1.3 (Pin_3)
- net USART1_RX: now also J11.3 (Pin_3)
- net USART1_TX: now also J11.2 (Pin_2)
- net at L1.1: now also C5.2, AP62200WU-1.2 (SW)
- net at R5.1: now also R4.2
- net at R3.2: now also C26.2, R5.2, AP62200WU-1.4 (FB)
- net at C5.1: now also AP62200WU-1.6 (BST)
- net NRST: now reaches R6.2, SW1.2 (B), U1.7 (NRST)
- net NRST: now also J1.1 (Pin_1)
- net at R4.1: now also R1.2
- new net: Q1.2 (G), R8.1
Other:
- moved on the sheet: C14, C2, C2A1, R6
